Commit message: URDF renewal

File: DHAL/DHAL.urdf (robot description, URDF)
Before this commit: robot DHAL, 14 links, 13 joints
Links:
- removed link L_Ankle
- removed link L_Hip_Pitch
- removed link R_Ankle
- removed link R_Hip_Pitch
- added link L_Ankle_Input_Left, mass 0.132288; visual mesh filename=Ankle_Link_Input.dae scale=1 1 1
- added link L_Ankle_Input_Right, mass 0.132288; visual mesh filename=Ankle_Link_Input_mir.dae scale=1 1 1
- added link L_Heel_Pitch_Left, mass 0.046696; visual mesh filename=Heel_Pitch.dae scale=1 1 1
- added link L_Heel_Pitch_Right, mass 0.046696; visual mesh filename=Heel_Pitch.dae scale=1 1 1
- added link L_Heel_Roll_Left, mass 0.116743; visual mesh filename=Ankle_Link_Short.dae scale=1 1 1
- added link L_Heel_Roll_Right, mass 0.144226; visual mesh filename=Ankle_Link_Long.dae scale=1 1 1
- added link L_Hip_to_Thigh, mass 0.260453; collision cylinder length=0.1 radius=0.09; visual mesh filename=Hip_to_Thigh.dae scale=1 1 1
- added link L_Knee_Input, mass 0.335783; visual mesh filename=Knee_Link_Input.dae scale=1 1 1
- added link L_Knee_Link, mass 0.203531; visual mesh filename=Knee_Link.dae scale=1 1 1
- added link L_Universal, mass 0.209567; visual mesh filename=Ankle_Universal.dae scale=1 1 1
- added link R_Ankle_Input_Left, mass 0.132288; visual mesh filename=Ankle_Link_Input.dae scale=1 1 1
- added link R_Ankle_Input_Right, mass 0.132288; visual mesh filename=Ankle_Link_Input_mir.dae scale=1 1 1
- added link R_Heel_Pitch_Left, mass 0.046696; visual mesh filename=Heel_Pitch.dae scale=1 1 1
- added link R_Heel_Pitch_Right, mass 0.046696; visual mesh filename=Heel_Pitch.dae scale=1 1 1
- added link R_Heel_Roll_Left, mass 0.144226; visual mesh filename=Ankle_Link_Long.dae scale=1 1 1
- added link R_Heel_Roll_Right, mass 0.116743; visual mesh filename=Ankle_Link_Short.dae scale=1 1 1
- added link R_Hip_to_Thigh, mass 0.260453; collision cylinder length=0.1 radius=0.09; visual mesh filename=Hip_to_Thigh_mir.dae scale=1 1 1
- added link R_Knee_Input, mass 0.335783; visual mesh filename=Knee_Link_Input_mir.dae scale=1 1 1
- added link R_Knee_Link, mass 0.203531; visual mesh filename=Knee_Link.dae scale=1 1 1
- added link R_Universal, mass 0.209567; visual mesh filename=Ankle_Universal.dae scale=1 1 1
- link L_Calf: mass 4.005008 -> 3.386071
- link L_Foot: mass 0.781383 -> 0.571816; geometry collision box size=0.18 0.08 0.02; collision cylinder length=0.02 radius=0.04
- link L_Thigh: mass 7.267508 -> 6.727728
- link Pelvis: mass 4.67 -> 4.775304
- link R_Calf: mass 4.005008 -> 3.386071
- link R_Foot: mass 0.781383 -> 0.571816; geometry collision box size=0.18 0.08 0.02; collision cylinder length=0.02 radius=0.04
- link R_Thigh: mass 7.267508 -> 6.727728
- link Torso: mass 12 -> 10.860955; geometry collision box size=0.14 0.242 0.374; visual mesh filename=Torso.dae scale=1 1 1
Joints:
- added joint L_ankle_input_left_joint: type revolute, parent L_Calf, child L_Ankle_Input_Left, origin xyz=-0.008 0.0255 -0.20464 rpy=0 0 0, axis 0 1 0, limit effort=150.0 velocity=10.0
- added joint L_ankle_input_right_joint: type revolute, parent L_Calf, child L_Ankle_Input_Right, origin xyz=-0.008 -0.0255 -0.08964 rpy=0 0 0, axis 0 1 0, limit effort=150.0 velocity=10.0
- added joint L_heel_pitch_left_joint: type revolute, parent L_Foot, child L_Heel_Pitch_Left, origin xyz=-0.06401 0.04 0.01129 rpy=0 0 0, axis 0 1 0
- added joint L_heel_pitch_right_joint: type revolute, parent L_Foot, child L_Heel_Pitch_Right, origin xyz=-0.06401 -0.04 0.01129 rpy=0 0 0, axis 0 1 0
- added joint L_heel_roll_left_joint: type revolute, parent L_Heel_Pitch_Left, child L_Heel_Roll_Left, origin xyz=0 0 0 rpy=0 0 0, axis 1 0 0
- added joint L_heel_roll_right_joint: type revolute, parent L_Heel_Pitch_Right, child L_Heel_Roll_Right, origin xyz=0 0 0 rpy=0 0 0, axis 1 0 0
- added joint L_knee_input_joint: type revolute, parent L_Thigh, child L_Knee_Input, origin xyz=0 0.1342 0 rpy=0 0 0, axis 0 1 0, limit effort=600.0 velocity=10.0
- added joint L_knee_link_joint: type revolute, parent L_Knee_Input, child L_Knee_Link, origin xyz=0.06 0.0165 0 rpy=0 0 0, axis 0 1 0
- added joint R_ankle_input_left_joint: type revolute, parent R_Calf, child R_Ankle_Input_Left, origin xyz=-0.008 0.0255 -0.08964 rpy=0 0 0, axis 0 1 0, limit effort=150.0 velocity=10.0
- added joint R_ankle_input_right_joint: type revolute, parent R_Calf, child R_Ankle_Input_Right, origin xyz=-0.008 -0.0255 -0.20464 rpy=0 0 0, axis 0 1 0, limit effort=150.0 velocity=10.0
- added joint R_heel_pitch_left_joint: type revolute, parent R_Foot, child R_Heel_Pitch_Left, origin xyz=-0.06401 0.04 0.01129 rpy=0 0 0, axis 0 1 0
- added joint R_heel_pitch_right_joint: type revolute, parent R_Foot, child R_Heel_Pitch_Right, origin xyz=-0.06401 -0.04 0.01129 rpy=0 0 0, axis 0 1 0
- added joint R_heel_roll_left_joint: type revolute, parent R_Heel_Pitch_Left, child R_Heel_Roll_Left, origin xyz=0 0 0 rpy=0 0 0, axis 1 0 0
- added joint R_heel_roll_right_joint: type revolute, parent R_Heel_Pitch_Right, child R_Heel_Roll_Right, origin xyz=0 0 0 rpy=0 0 0, axis 1 0 0
- added joint R_knee_input_joint: type revolute, parent R_Thigh, child R_Knee_Input, origin xyz=0 -0.1342 0 rpy=0 0 0, axis 0 1 0, limit effort=600.0 velocity=10.0
- added joint R_knee_link_joint: type revolute, parent R_Knee_Input, child R_Knee_Link, origin xyz=0.06 -0.0165 0 rpy=0 0 0, axis 0 1 0
- joint L_ankle_pitch_joint: child L_Ankle -> L_Universal; limit lower=-1.22173 upper=0.349066 effort=150.0 velocity=10.0 -> lower=-0.872665 upper=0.698132
- joint L_ankle_roll_joint: limit lower=-0.523599 upper=0.523599 effort=150.0 velocity=10.0 -> lower=-0.523599 upper=0.523599; parent L_Ankle -> L_Universal
- joint L_hip_pitch_joint: parent L_Hip_Pitch -> L_Hip_to_Thigh
- joint L_hip_roll_joint: child L_Hip_Pitch -> L_Hip_to_Thigh
- joint L_knee_joint: limit lower=0.0872665 upper=2.35619 effort=600.0 velocity=10.0 -> lower=0.0872665 upper=2.35619
- joint R_ankle_pitch_joint: child R_Ankle -> R_Universal; limit lower=-1.22173 upper=0.349066 effort=150.0 velocity=10.0 -> lower=-0.872665 upper=0.698132
- joint R_ankle_roll_joint: limit lower=-0.523599 upper=0.523599 effort=150.0 velocity=10.0 -> lower=-0.523599 upper=0.523599; parent R_Ankle -> R_Universal
- joint R_hip_pitch_joint: parent R_Hip_Pitch -> R_Hip_to_Thigh
- joint R_hip_roll_joint: child R_Hip_Pitch -> R_Hip_to_Thigh; limit lower=-0.785398 upper=0.349066 effort=360.0 velocity=10.0 -> lower=-0.349066 upper=0.785398 effort=360.0 velocity=10.0
- joint R_hip_yaw_joint: limit lower=-1.57079632679 upper=0.785398 effort=360.0 velocity=10.0 -> lower=-0.785398 upper=1.57079632679 effort=360.0 velocity=10.0
- joint R_knee_joint: limit lower=0.0872665 upper=2.35619 effort=600.0 velocity=10.0 -> lower=0.0872665 upper=2.35619
- joint waist_yaw_joint: limit lower=-0.785398 upper=0.785398 effort=360.0 velocity=10.0 -> lower=-1.57080 upper=-1.57080 effort=360.0 velocity=10.0; origin xyz=0.04 0 0.052 rpy=0 0 0 -> xyz=0.04 0.0 0.052 rpy=0 0 0

Commit message: remove URDF_ head and change torso movement range

File: DHAL/DHAL.urdf (robot description, URDF)
Before this commit: robot DHAL, 30 links, 29 joints
Joints:
- joint waist_yaw_joint: limit lower=-1.57080 upper=-1.57080 effort=360.0 velocity=10.0 -> lower=-1.57080 upper=1.57080 effort=360.0 velocity=10.0

Commit message: renewal 13 DOF URDF

File: DHAL/DHAL.urdf (robot description, URDF)
Before this commit: robot DHAL, 30 links, 29 joints
Links:
- removed link L_Ankle_Input_Left
- removed link L_Ankle_Input_Right
- removed link L_Heel_Pitch_Left
- removed link L_Heel_Pitch_Right
- removed link L_Heel_Roll_Left
- removed link L_Heel_Roll_Right
- removed link L_Knee_Input
- removed link L_Knee_Link
- removed link R_Ankle_Input_Left
- removed link R_Ankle_Input_Right
- removed link R_Heel_Pitch_Left
- removed link R_Heel_Pitch_Right
- removed link R_Heel_Roll_Left
- removed link R_Heel_Roll_Right
- removed link R_Knee_Input
- removed link R_Knee_Link
- link L_Calf: mass 3.386071 -> 4.005008; geometry collision box size=0.1 0.05 0.30; visual mesh filename=URDF_Calf_Left.dae scale=1 1 1
- link L_Foot: geometry collision box size=0.18 0.08 0.02; collision cylinder length=0.02 radius=0.04
- link L_Hip: mass 2.204506 -> 2.157752; geometry collision cylinder length=0.08 radius=0.06; visual mesh filename=URDF_Hip.dae scale=1 1 1
- link L_Hip_to_Thigh: mass 0.260453 -> 0.794453; geometry collision cylinder length=0.19 radius=0.09; visual mesh filename=URDF_Hip_to_Thigh_Left.dae scale=1 1 1
- link L_Thigh: mass 6.727728 -> 7.063633; geometry visual mesh filename=URDF_Thigh_Left.dae scale=1 1 1
- link L_Universal: geometry visual mesh filename=URDF_Universal.dae scale=1 1 1
- link Pelvis: mass 4.775304 -> 4.509446; geometry collision box size=0.11 0.32 0.09; visual mesh filename=URDF_Pelvis.dae scale=1 1 1
- link R_Calf: mass 3.386071 -> 4.005008; geometry collision box size=0.1 0.05 0.30; visual mesh filename=URDF_Calf_Right.dae scale=1 1 1
- link R_Foot: geometry collision box size=0.18 0.08 0.02; collision cylinder length=0.02 radius=0.04
- link R_Hip: mass 2.204506 -> 2.157752; geometry collision cylinder length=0.08 radius=0.06; visual mesh filename=URDF_Hip.dae scale=1 1 1
- link R_Hip_to_Thigh: mass 0.260453 -> 0.794453; geometry collision cylinder length=0.19 radius=0.09; visual mesh filename=URDF_Hip_to_Thigh_Right.dae scale=1 1 1
- link R_Thigh: mass 6.727728 -> 7.063633; geometry visual mesh filename=URDF_Thigh_Right.dae scale=1 1 1
- link R_Universal: geometry visual mesh filename=URDF_Universal.dae scale=1 1 1
- link Torso: mass 10.860955 -> 10.742786; geometry collision box size=0.14 0.242 0.374; visual mesh filename=URDF_Torso.dae scale=1 1 1
Joints:
- removed joint L_ankle_input_left_joint
- removed joint L_ankle_input_right_joint
- removed joint L_heel_pitch_left_joint
- removed joint L_heel_pitch_right_joint
- removed joint L_heel_roll_left_joint
- removed joint L_heel_roll_right_joint
- removed joint L_knee_input_joint
- removed joint L_knee_link_joint
- removed joint R_ankle_input_left_joint
- removed joint R_ankle_input_right_joint
- removed joint R_heel_pitch_left_joint
- removed joint R_heel_pitch_right_joint
- removed joint R_heel_roll_left_joint
- removed joint R_heel_roll_right_joint
- removed joint R_knee_input_joint
- removed joint R_knee_link_joint
- joint L_ankle_pitch_joint: limit lower=-0.872665 upper=0.698132 -> lower=-0.872665 upper=0.698132 effort=360.0 velocity=10.0
- joint L_ankle_roll_joint: limit lower=-0.523599 upper=0.523599 -> lower=-0.523599 upper=0.523599 effort=360.0 velocity=10.0
- joint L_hip_pitch_joint: limit lower=-1.57079632679 upper=1.57079632679 effort=600.0 velocity=10.0 -> lower=-1.570796 upper=1.570796 effort=600.0 velocity=10.0; origin xyz=0.096 -0.0451 0 rpy=0 0 0 -> xyz=0.096 -0.0451 0 rpy=0 -0.785398 0
- joint L_hip_roll_joint: limit lower=-0.349066 upper=0.785398 effort=360.0 velocity=10.0 -> lower=-1.570796 upper=1.570796 effort=360.0 velocity=10.0
- joint L_hip_yaw_joint: limit lower=-0.785398 upper=1.57079632679 effort=360.0 velocity=10.0 -> lower=-1.570796 upper=1.570796 effort=360.0 velocity=10.0; origin xyz=0.0 0.1 -0.0492 rpy=0 0 0 -> xyz=0.0 0.1 0.0 rpy=0 0.785398 0
- joint L_knee_joint: limit lower=0.0872665 upper=2.35619 -> lower=0.0872665 upper=2.35619 effort=600.0 velocity=10.0
- joint R_ankle_pitch_joint: limit lower=-0.872665 upper=0.698132 -> lower=-0.872665 upper=0.698132 effort=360.0 velocity=10.0
- joint R_ankle_roll_joint: limit lower=-0.523599 upper=0.523599 -> lower=-0.523599 upper=0.523599 effort=360.0 velocity=10.0
- joint R_hip_pitch_joint: limit lower=-1.57079632679 upper=1.57079632679 effort=600.0 velocity=10.0 -> lower=-1.570796 upper=1.570796 effort=600.0 velocity=10.0; origin xyz=0.096 0.0451 0 rpy=0 0 0 -> xyz=0.096 0.0451 0 rpy=0 -0.785398 0
- joint R_hip_roll_joint: limit lower=-0.349066 upper=0.785398 effort=360.0 velocity=10.0 -> lower=-1.570796 upper=1.570796 effort=360.0 velocity=10.0
- joint R_hip_yaw_joint: limit lower=-0.785398 upper=1.57079632679 effort=360.0 velocity=10.0 -> lower=-1.570796 upper=1.570796 effort=360.0 velocity=10.0; origin xyz=0.0 -0.1 -0.0492 rpy=0 0 0 -> xyz=0.0 -0.1 0 rpy=0 0.785398 0
- joint R_knee_joint: limit lower=0.0872665 upper=2.35619 -> lower=0.0872665 upper=2.35619 effort=600.0 velocity=10.0
- joint waist_yaw_joint: limit lower=-1.57080 upper=1.57080 effort=360.0 velocity=10.0 -> lower=-1.570796 upper=1.570796 effort=360.0 velocity=10.0; origin xyz=0.04 0.0 0.052 rpy=0 0 0 -> xyz=0.065 0.0 0.096 rpy=0 0 0
